Commit message: Simplify intertials to work properly with the simulation.

File: xarm_description/urdf/common/common.link.xacro (robot description, xacro)
@@ -1,4 +1,11 @@
 <?xml version="1.0"?>
 <robot xmlns:xacro="http://ros.org/wiki/xacro">
+  <xacro:macro name="default_inertial">
+    <inertial>
+      <mass value="0.01"/>
+      <origin xyz="0 0 0"/>
+      <inertia ixx="0.001" ixy="0.0" ixz="0.0" iyy="0.001" iyz="0.0" izz="0.001" />
+    </inertial>
+  </xacro:macro>
   <xacro:macro name="common_link_inertial" params="link_inertial_params origin_rpy:='0 0 0'">
     <inertial>

File: xarm_description/urdf/xarm5/xarm5.urdf.xacro (robot description, xacro)
@@ -37,5 +37,6 @@
     <xacro:property name="kinematics_params" value="${kinematics_config['kinematics']}"/>
     <link name="${prefix}link_base">
-      <inertial>
+      <xacro:default_inertial />
+      <!--<inertial>
         <origin xyz="-0.00218 -0.00023 0.08604" rpy="0 0 0" />
         <mass value="1.95" />
@@ -43,5 +44,5 @@
           ixx="0.004805" ixy="-8.33E-06" ixz="0.00026847"
           iyy="0.0050349" iyz="7.23E-06" izz="0.0025418" />
-      </inertial>
+      </inertial>-->
       <xacro:common_link_visual
         mesh_filename="xarm5/visual/link_base"
@@ -55,7 +56,8 @@
     </link>
     <link name="${prefix}link1">
-      <xacro:common_link_inertial
+      <xacro:default_inertial />
+      <!--<xacro:common_link_inertial
         link_inertial_params="${inertial_params['link1']}"
-        origin_rpy="0 0 0"/>
+        origin_rpy="0 0 0"/>-->
       <xacro:common_link_visual
         mesh_filename="xarm5/visual/link1"
@@ -82,7 +84,8 @@
     </joint>
     <link name="${prefix}link2">
-      <xacro:common_link_inertial
+      <xacro:default_inertial />
+      <!--<xacro:common_link_inertial
         link_inertial_params="${inertial_params['link2']}"
-        origin_rpy="0 0 0"/>
+        origin_rpy="0 0 0"/>-->
       <xacro:common_link_visual
         mesh_filename="xarm5/visual/link2"
@@ -109,7 +112,8 @@
     </joint>
     <link name="${prefix}link3">
-      <xacro:common_link_inertial
+      <xacro:default_inertial />
+      <!--<xacro:common_link_inertial
         link_inertial_params="${inertial_params['link3']}"
-        origin_rpy="0 0 0"/>
+        origin_rpy="0 0 0"/>-->
       <xacro:common_link_visual
         mesh_filename="xarm5/visual/link3"
@@ -136,7 +140,8 @@
     </joint>
     <link name="${prefix}link4">
-      <xacro:common_link_inertial
+      <xacro:default_inertial />
+      <!--<xacro:common_link_inertial
         link_inertial_params="${inertial_params['link4']}"
-        origin_rpy="0 0 0"/>
+        origin_rpy="0 0 0"/>-->
       <xacro:common_link_visual
         mesh_filename="xarm5/visual/link4"
@@ -163,7 +168,8 @@
     </joint>
     <link name="${prefix}link5">
-      <xacro:common_link_inertial
+      <xacro:default_inertial />
+      <!--<xacro:common_link_inertial
         link_inertial_params="${inertial_params['link5']}"
-        origin_rpy="0 0 0"/>
+        origin_rpy="0 0 0"/>-->
       <xacro:common_link_visual
         mesh_filename="${end_tool_visual_filename}"
